Commit message: Changed urdfs to add a center gripper frame

File: franka_description/robots/hand.urdf.xacro (robot description, xacro)
@@ -1,5 +1,10 @@
 <?xml version="1.0" encoding="utf-8"?>
 <robot xmlns:xacro="http://www.ros.org/wiki/xacro" name="hand">
-  <xacro:include filename="hand.xacro"/>
-  <xacro:hand ns="panda"/>
+  <!-- Initialize gripper_center properties -->
+  <xacro:arg name="gripper_center" default="false" /> <!-- Default value -->
+  <xacro:property name="gripper_center" value="$(arg gripper_center)"/> <!-- Overload with launchfile argument -->
+  <xacro:arg name="gripper_center_xyz" default="0.0 0.0 0.10" /> <!-- Default value -->
+  <xacro:property name="gripper_center_xyz" value="$(arg gripper_center_xyz)"/> <!-- Overload with launchfile argument -->
+  <!-- Create the hand urdf -->
+  <xacro:hand ns="panda" gripper_center="${gripper_center}" gripper_center_xyz="${gripper_center_xyz}"/>
 </robot>

File: franka_description/robots/hand.xacro (robot description, xacro)
@@ -1,5 +1,5 @@
 <?xml version="1.0" encoding="utf-8"?>
 <robot xmlns:xacro="http://www.ros.org/wiki/xacro" name="hand">
-  <xacro:macro name="hand" params="connected_to:='' ns:='' rpy:='0 0 0' xyz:='0 0 0' ">
+  <xacro:macro name="hand" params="connected_to:='' ns:='' rpy:='0 0 0' xyz:='0 0 0' gripper_center:='false' gripper_center_xyz:='0.0 0.0 0.10'">
     <xacro:unless value="${connected_to == ''}">
       <joint name="${ns}_hand_joint" type="fixed">
@@ -9,4 +9,5 @@
       </joint>
     </xacro:unless>
+    <!-- Links -->
     <link name="${ns}_hand">
       <visual>
@@ -62,4 +63,5 @@
       </inertial>
     </link>
+    <!-- Joints -->
     <joint name="${ns}_finger_joint1" type="prismatic">
       <parent link="${ns}_hand"/>
@@ -77,4 +79,15 @@
       <mimic joint="${ns}_finger_joint1" />
     </joint>
+    <!-- Create gripper center virtual link and joint -->
+    <xacro:if value="${gripper_center}"> <!-- Only when gripper_center==True -->
+      <link name="${ns}_gripper_center">
+      </link>
+      <joint name="${ns}_gripper_center_joint" type="fixed">
+        <parent link="${ns}_hand"/>
+        <child link="${ns}_gripper_center"/>
+        <origin xyz="${gripper_center_xyz}" rpy="0 0 0"/>
+        <axis xyz="0 -1 0"/>
+      </joint>
+    </xacro:if>
   </xacro:macro>
 </robot>

File: franka_description/robots/panda_arm_hand.urdf.xacro (robot description, xacro)
@@ -1,11 +1,19 @@
 <?xml version="1.0" encoding="utf-8"?>
 <robot xmlns:xacro="http://www.ros.org/wiki/xacro" name="panda">
+  <!-- Initialize xacro parameters -->
   <xacro:arg name="robot_name" default="panda"/>
+  <!-- Initialize gripper_center properties -->
+  <xacro:arg name="gripper_center" default="false" />
+  <xacro:property name="gripper_center" value="$(arg gripper_center)"/>
+  <xacro:arg name="gripper_center_xyz" default="0.0 0.0 0.10" />
+  <xacro:property name="gripper_center_xyz" value="$(arg gripper_center_xyz)"/>
+  <!-- Include xacro files -->
   <xacro:include filename="$(find franka_description)/robots/panda_arm.xacro"/>
   <xacro:include filename="$(find franka_description)/robots/hand.xacro"/>
   <xacro:include filename="$(find franka_description)/robots/panda.gazebo.xacro"/>
   <xacro:include filename="$(find franka_description)/robots/panda.transmission.xacro"/>
+  <!-- Generate urdfs -->
   <xacro:panda_arm />
-  <xacro:hand ns="panda" rpy="0 0 ${-pi/4}" connected_to="panda_link8"/>
+  <xacro:hand ns="panda" rpy="0 0 ${-pi/4}" connected_to="panda_link8" gripper_center="${gripper_center}" gripper_center_xyz="${gripper_center_xyz}"/>
   <xacro:panda_gazebo robot_name="$(arg robot_name)" />
   <xacro:panda_transmission robot_name="$(arg robot_name)" />

Commit message: :sparkles: Adds virtual grip site link
In order to control the robot w.r.t. the center of the gripper a virtual grip site link and joint were added.

File: franka_description/robots/hand.urdf.xacro (robot description, xacro)
@@ -2,4 +2,9 @@
 <robot xmlns:xacro="http://www.ros.org/wiki/xacro" name="hand">
   <xacro:include filename="hand.xacro"/>
-  <xacro:hand ns="panda"/>
+  <!-- Initialize grip_site properties -->
+  <xacro:arg name="grip_site" default="false" /> <!-- Default value -->
+  <xacro:property name="grip_site" value="$(arg grip_site)" /> <!-- Overload with launchfile argument -->
+  <xacro:arg name="grip_site_xyz" default="0.0 0.0 0.10" /> <!-- Default value -->
+  <xacro:property name="grip_site_xyz" value="$(arg grip_site_xyz)" /> <!-- Overload with launchfile argument -->
+  <xacro:hand ns="panda" grip_site="${grip_site}" grip_site_xyz="${grip_site_xyz}" grip_site_rpy="${grip_site_rpy}" />
 </robot>

File: franka_description/robots/hand.xacro (robot description, xacro)
@@ -1,5 +1,5 @@
 <?xml version="1.0" encoding="utf-8"?>
 <robot xmlns:xacro="http://www.ros.org/wiki/xacro" name="hand">
-  <xacro:macro name="hand" params="connected_to:='' ns:='' rpy:='0 0 0' xyz:='0 0 0' ">
+  <xacro:macro name="hand" params="connected_to:='' ns:='' rpy:='0 0 0' xyz:='0 0 0' grip_site:='false' grip_site_xyz:='0.0 0.0 0.10' grip_site_rpy:='0.0 0.0 0.0'">
     <xacro:unless value="${connected_to == ''}">
       <joint name="${ns}_hand_joint" type="fixed">
@@ -82,4 +82,15 @@
       <limit effort="20" lower="0.0" upper="0.04" velocity="0.2"/>
     </joint>
+    <!-- Add virtual grip site link -->
+    <xacro:if value="${grip_site}">
+      <!-- Only when grip_site==True -->
+      <link name="${ns}_grip_site"/>
+      <joint name="${ns}_grip_site_joint" type="fixed">
+        <parent link="${ns}_hand" />
+        <child link="${ns}_grip_site" />
+        <origin xyz="${grip_site_xyz}" rpy="${grip_site_rpy}" />
+        <axis xyz="0 -1 0" />
+      </joint>
+    </xacro:if>
   </xacro:macro>
 </robot>

File: franka_description/robots/panda_arm_hand.urdf.xacro (robot description, xacro)
@@ -3,4 +3,11 @@
   <xacro:include filename="$(find franka_description)/robots/panda_arm.xacro"/>
   <xacro:include filename="$(find franka_description)/robots/hand.xacro"/>
+  <!-- Initialize grip_site properties -->
+  <xacro:arg name="grip_site" default="false" />
+  <xacro:property name="grip_site" value="$(arg grip_site)" />
+  <xacro:arg name="grip_site_xyz" default="0.0 0.0 0.10" />
+  <xacro:property name="grip_site_xyz" value="$(arg grip_site_xyz)" />
+  <xacro:arg name="grip_site_rpy" default="0.0 0.0 0.0" />
+  <xacro:property name="grip_site_rpy" value="$(arg grip_site_rpy)" />
   <!-- for simulation -->
   <xacro:include filename="$(find franka_description)/robots/panda.gazebo.xacro"/>
@@ -8,5 +15,5 @@
   <!-- end for simulation -->
   <xacro:panda_arm />
-  <xacro:hand ns="panda" rpy="0 0 ${-pi/4}" connected_to="panda_link8"/>
+  <xacro:hand ns="panda" rpy="0 0 ${-pi/4}" connected_to="panda_link8" grip_site="${grip_site}" grip_site_xyz="${grip_site_xyz}" grip_site_rpy="${grip_site_rpy}" />
   <!-- for simulation -->
   <xacro:arg name="robot_name" default="panda"/>

Commit message: Full split between hand and arm xacro files.

File: franka_description/robots/hand.urdf.xacro (robot description, xacro)
@@ -2,4 +2,12 @@
 <robot xmlns:xacro="http://www.ros.org/wiki/xacro" name="hand">
   <xacro:include filename="hand.xacro"/>
-  <xacro:hand ns="panda" safety_distance="0.03"/>
+  <!-- for simulation -->
+  <xacro:include filename="$(find franka_description)/robots/panda.gazebo.xacro"/>
+  <xacro:include filename="$(find franka_description)/robots/panda.control.xacro"/>
+  <!-- end for simulation -->
+  <xacro:hand ns="panda" rpy="0 0 ${-pi/4}" connected_to="panda_link8" safety_distance="0.03"/>
+  <!-- for simulation -->
+  <xacro:hand_gazebo arm_id="$(arg arm_id)"/>
+  <xacro:hand_control arm_id="$(arg arm_id)"/>
+  <!-- end for simulation -->
 </robot>

File: franka_description/robots/panda.control.xacro (robot description, xacro)
@@ -1,31 +1,31 @@
 <?xml version="1.0"?>
 <robot xmlns:xacro="http://www.ros.org/wiki/xacro">
-    <xacro:macro name="panda_control" params="arm_id load_hand">
-        <xacro:macro name="arm_control" params="transmission joint motor">
-            <transmission name="${transmission}">
-                <type>transmission_interface/SimpleTransmission</type>
-                <joint name="${joint}">
-                    <hardwareInterface>hardware_interface/PositionJointInterface</hardwareInterface>
-                </joint>
-                <actuator name="${motor}">
-                    <hardwareInterface>hardware_interface/PositionJointInterface</hardwareInterface>
-                    <mechanicalReduction>1</mechanicalReduction>
-                </actuator>
-            </transmission>
-        </xacro:macro>
-        <xacro:arm_control transmission="${arm_id}_tran_1" joint="${arm_id}_joint1" motor="${arm_id}_motor_1"/>
-        <xacro:arm_control transmission="${arm_id}_tran_2" joint="${arm_id}_joint2" motor="${arm_id}_motor_2"/>
-        <xacro:arm_control transmission="${arm_id}_tran_3" joint="${arm_id}_joint3" motor="${arm_id}_motor_3"/>
-        <xacro:arm_control transmission="${arm_id}_tran_4" joint="${arm_id}_joint4" motor="${arm_id}_motor_4"/>
-        <xacro:arm_control transmission="${arm_id}_tran_5" joint="${arm_id}_joint5" motor="${arm_id}_motor_5"/>
-        <xacro:arm_control transmission="${arm_id}_tran_6" joint="${arm_id}_joint6" motor="${arm_id}_motor_6"/>
-        <xacro:arm_control transmission="${arm_id}_tran_7" joint="${arm_id}_joint7" motor="${arm_id}_motor_7"/>
-        <xacro:if value="${load_hand}">
-            <xacro:arm_control transmission="${arm_id}_leftfinger" joint="${arm_id}_finger_joint1" motor="${arm_id}_finger_joint1"/>
-            <xacro:arm_control transmission="${arm_id}_rightfinger" joint="${arm_id}_finger_joint2" motor="${arm_id}_finger_joint2"/>
-        </xacro:if>
-        <gazebo>
-            <plugin name="gazebo_ros_control" filename="libgazebo_ros_control.so"/>
-        </gazebo>
+    <xacro:macro name="joint_control" params="transmission joint motor">
+        <transmission name="${transmission}">
+            <type>transmission_interface/SimpleTransmission</type>
+            <joint name="${joint}">
+                <hardwareInterface>hardware_interface/PositionJointInterface</hardwareInterface>
+            </joint>
+            <actuator name="${motor}">
+                <hardwareInterface>hardware_interface/PositionJointInterface</hardwareInterface>
+                <mechanicalReduction>1</mechanicalReduction>
+            </actuator>
+        </transmission>
     </xacro:macro>
+    <xacro:macro name="arm_control" params="arm_id">
+        <xacro:joint_control transmission="${arm_id}_tran_1" joint="${arm_id}_joint1" motor="${arm_id}_motor_1"/>
+        <xacro:joint_control transmission="${arm_id}_tran_2" joint="${arm_id}_joint2" motor="${arm_id}_motor_2"/>
+        <xacro:joint_control transmission="${arm_id}_tran_3" joint="${arm_id}_joint3" motor="${arm_id}_motor_3"/>
+        <xacro:joint_control transmission="${arm_id}_tran_4" joint="${arm_id}_joint4" motor="${arm_id}_motor_4"/>
+        <xacro:joint_control transmission="${arm_id}_tran_5" joint="${arm_id}_joint5" motor="${arm_id}_motor_5"/>
+        <xacro:joint_control transmission="${arm_id}_tran_6" joint="${arm_id}_joint6" motor="${arm_id}_motor_6"/>
+        <xacro:joint_control transmission="${arm_id}_tran_7" joint="${arm_id}_joint7" motor="${arm_id}_motor_7"/>
+    </xacro:macro>
+    <xacro:macro name="hand_control" params="arm_id">
+        <xacro:joint_control transmission="${arm_id}_leftfinger" joint="${arm_id}_finger_joint1" motor="${arm_id}_finger_joint1"/>
+        <xacro:joint_control transmission="${arm_id}_rightfinger" joint="${arm_id}_finger_joint2" motor="${arm_id}_finger_joint2"/>
+    </xacro:macro>
+    <gazebo>
+        <plugin name="gazebo_ros_control" filename="libgazebo_ros_control.so"/>
+    </gazebo>
 </robot>

File: franka_description/robots/panda.gazebo.xacro (robot description, xacro)
@@ -1,6 +1,6 @@
 <?xml version='1.0' encoding='utf-8'?>
 <robot xmlns:xacro="http://www.ros.org/wiki/xacro">
-    <xacro:macro name="panda_gazebo" params="arm_id">
-        <xacro:macro name="arm_gazebo" params="link">
+    <xacro:macro name="arm_gazebo" params="arm_id">
+        <xacro:macro name="arm_link_gazebo" params="link">
             <gazebo reference="${link}">
                 <material>Gazebo/White</material>
@@ -9,5 +9,16 @@
             </gazebo>
         </xacro:macro>
-        <xacro:macro name="hand_gazebo" params="link">
+        <xacro:arm_link_gazebo link="${arm_id}_link0"/>
+        <xacro:arm_link_gazebo link="${arm_id}_link1"/>
+        <xacro:arm_link_gazebo link="${arm_id}_link2"/>
+        <xacro:arm_link_gazebo link="${arm_id}_link3"/>
+        <xacro:arm_link_gazebo link="${arm_id}_link4"/>
+        <xacro:arm_link_gazebo link="${arm_id}_link5"/>
+        <xacro:arm_link_gazebo link="${arm_id}_link6"/>
+        <xacro:arm_link_gazebo link="${arm_id}_link7"/>
+        <xacro:arm_link_gazebo link="${arm_id}_link8"/>
+    </xacro:macro>
+    <xacro:macro name="hand_gazebo" params="arm_id">
+        <xacro:macro name="hand_link_gazebo" params="link">
             <gazebo reference="${link}">
                 <material>Gazebo/Grey</material>
@@ -16,16 +27,7 @@
             </gazebo>
         </xacro:macro>
-        <xacro:arm_gazebo link="${arm_id}_link0"/>
-        <xacro:arm_gazebo link="${arm_id}_link1"/>
-        <xacro:arm_gazebo link="${arm_id}_link2"/>
-        <xacro:arm_gazebo link="${arm_id}_link3"/>
-        <xacro:arm_gazebo link="${arm_id}_link4"/>
-        <xacro:arm_gazebo link="${arm_id}_link5"/>
-        <xacro:arm_gazebo link="${arm_id}_link6"/>
-        <xacro:hand_gazebo link="${arm_id}_link7"/>
-        <xacro:hand_gazebo link="${arm_id}_link8"/>
-        <xacro:hand_gazebo link="${arm_id}_hand"/>
-        <xacro:hand_gazebo link="${arm_id}_rightfinger"/>
-        <xacro:hand_gazebo link="${arm_id}_leftfinger"/>
+        <xacro:hand_link_gazebo link="${arm_id}_hand"/>
+        <xacro:hand_link_gazebo link="${arm_id}_rightfinger"/>
+        <xacro:hand_link_gazebo link="${arm_id}_leftfinger"/>
     </xacro:macro>
 </robot>

File: franka_description/robots/panda_arm.urdf.xacro (robot description, xacro)
@@ -1,4 +1,5 @@
 <?xml version='1.0' encoding='utf-8'?>
 <robot xmlns:xacro="http://www.ros.org/wiki/xacro" name="panda">
+  <xacro:arg name="arm_id" default="panda"/>
   <xacro:include filename="$(find franka_description)/robots/panda_arm.xacro" />
   <!-- for simulation -->
@@ -6,9 +7,8 @@
   <xacro:include filename="$(find franka_description)/robots/panda.control.xacro"/>
   <!-- end for simulation -->
-  <xacro:panda_arm xyz="0 0 0" rpy="0 0 0" connected_to="world" arm_id="panda" safety_distance="0.03"/>
+  <xacro:panda_arm xyz="0 0 0" rpy="0 0 0" connected_to="world" arm_id="$(arg arm_id)" safety_distance="0.03"/>
   <!-- for simulation -->
-  <xacro:arg name="robot_name" default="panda"/>
-  <xacro:panda_gazebo robot_name="$(arg robot_name)" />
-  <xacro:panda_transmission robot_name="$(arg robot_name)" load_hand="false" />
+  <xacro:arm_gazebo arm_id="$(arg arm_id)"/>
+  <xacro:arm_control arm_id="$(arg arm_id)"/>
   <!-- end for simulation -->
 </robot>

File: franka_description/robots/panda_arm_hand.urdf.xacro (robot description, xacro)
@@ -1,16 +1,5 @@
 <?xml version="1.0" encoding="utf-8"?>
 <robot xmlns:xacro="http://www.ros.org/wiki/xacro" name="panda">
-  <xacro:include filename="$(find franka_description)/robots/panda_arm.xacro"/>
-  <xacro:include filename="$(find franka_description)/robots/hand.xacro"/>
-  <!-- for simulation -->
-  <xacro:include filename="$(find franka_description)/robots/panda.gazebo.xacro"/>
-  <xacro:include filename="$(find franka_description)/robots/panda.control.xacro"/>
-  <!-- end for simulation -->
-  <link name="world" />
-  <xacro:panda_arm xyz="0 0 0" rpy="0 0 0" connected_to="world" arm_id="panda" safety_distance="0.03"/>
-  <xacro:hand ns="panda" rpy="0 0 ${-pi/4}" connected_to="panda_link8" safety_distance="0.03"/>
-  <!-- for simulation -->
-  <xacro:panda_gazebo arm_id="panda"/>
-  <xacro:panda_control arm_id="panda" load_hand="true" />
-  <!-- end for simulation -->
+  <xacro:include filename="$(find franka_description)/robots/panda_arm.urdf.xacro"/>
+  <xacro:include filename="$(find franka_description)/robots/hand.urdf.xacro"/>
 </robot>
