Commit message: Parameterize collisions for whether to use cylinder or mesh model.

File: franka_description/robots/hand.urdf.xacro (robot description, xacro)
@@ -1,4 +1,5 @@
 <?xml version="1.0" encoding="utf-8"?>
 <robot xmlns:xacro="http://www.ros.org/wiki/xacro" name="hand">
+  <xacro:arg name="use_cylinder_collision_model" default="true"/>
   <xacro:include filename="hand.xacro"/>
   <!-- for simulation -->
@@ -6,5 +7,6 @@
   <xacro:include filename="$(find franka_description)/robots/panda.control.xacro"/>
   <!-- end for simulation -->
-  <xacro:hand ns="panda" rpy="0 0 ${-pi/4}" connected_to="panda_link8" safety_distance="0.03"/>
+  <xacro:hand ns="panda" rpy="0 0 ${-pi/4}" connected_to="panda_link8" safety_distance="0.03"
+    use_cylinder_collision_model="$(arg use_cylinder_collision_model)"/>
   <!-- for simulation -->
   <xacro:hand_gazebo arm_id="$(arg arm_id)"/>

File: franka_description/robots/hand.xacro (robot description, xacro)
@@ -2,5 +2,6 @@
 <robot xmlns:xacro="http://www.ros.org/wiki/xacro" name="hand">
   <!-- safety_distance: Minimum safety distance in [m] by which the collision volumes are expanded and which is enforced during robot motions -->
-  <xacro:macro name="hand" params="connected_to:='' ns:='' rpy:='0 0 0' xyz:='0 0 0' safety_distance:=0">
+  <xacro:macro name="hand" params="connected_to:='' ns:='' rpy:='0 0 0' xyz:='0 0 0' safety_distance:=0
+    use_cylinder_collision_model:='true'">
     <xacro:unless value="${connected_to == ''}">
       <joint name="${ns}_hand_joint" type="fixed">
@@ -16,40 +17,49 @@
         </geometry>
       </visual>
-      <collision>
-        <origin xyz="0 0 0.04" rpy="0 ${pi/2} ${pi/2}"/>
-        <geometry>
-          <cylinder radius="${0.04+safety_distance}" length="0.1" />
-        </geometry>
-      </collision>
-      <collision>
-        <origin xyz="0 -0.05 0.04" rpy="0 0 0"/>
-        <geometry>
-          <sphere radius="${0.04+safety_distance}"  />
-        </geometry>
-      </collision>
-      <collision>
-        <origin xyz="0 0.05 0.04" rpy="0 0 0"/>
-        <geometry>
-          <sphere radius="${0.04+safety_distance}"  />
-        </geometry>
-      </collision>
-      <collision>
-        <origin xyz="0 0 0.1" rpy="0 ${pi/2} ${pi/2}"/>
-        <geometry>
-          <cylinder radius="${0.02+safety_distance}" length="0.1" />
-        </geometry>
-      </collision>
-      <collision>
-        <origin xyz="0 -0.05 0.1" rpy="0 0 0"/>
-        <geometry>
-          <sphere radius="${0.02+safety_distance}"  />
-        </geometry>
-      </collision>
-      <collision>
-        <origin xyz="0 0.05 0.1" rpy="0 0 0"/>
-        <geometry>
-          <sphere radius="${0.02+safety_distance}"  />
-        </geometry>
-      </collision>
+      <xacro:if value="${use_cylinder_collision_model}">
+        <collision>
+          <origin xyz="0 0 0.04" rpy="0 ${pi/2} ${pi/2}"/>
+          <geometry>
+            <cylinder radius="${0.04+safety_distance}" length="0.1" />
+          </geometry>
+        </collision>
+        <collision>
+          <origin xyz="0 -0.05 0.04" rpy="0 0 0"/>
+          <geometry>
+            <sphere radius="${0.04+safety_distance}"  />
+          </geometry>
+        </collision>
+        <collision>
+          <origin xyz="0 0.05 0.04" rpy="0 0 0"/>
+          <geometry>
+            <sphere radius="${0.04+safety_distance}"  />
+          </geometry>
+        </collision>
+        <collision>
+          <origin xyz="0 0 0.1" rpy="0 ${pi/2} ${pi/2}"/>
+          <geometry>
+            <cylinder radius="${0.02+safety_distance}" length="0.1" />
+          </geometry>
+        </collision>
+        <collision>
+          <origin xyz="0 -0.05 0.1" rpy="0 0 0"/>
+          <geometry>
+            <sphere radius="${0.02+safety_distance}"  />
+          </geometry>
+        </collision>
+        <collision>
+          <origin xyz="0 0.05 0.1" rpy="0 0 0"/>
+          <geometry>
+            <sphere radius="${0.02+safety_distance}"  />
+          </geometry>
+        </collision>
+      </xacro:if>
+      <xacro:unless value="${use_cylinder_collision_model}">
+        <collision>
+          <geometry>
+            <mesh filename="package://franka_description/meshes/collision/hand.stl"/>
+          </geometry>
+        </collision>
+      </xacro:unless>
       <!-- for simulation -->
       <inertial>
@@ -66,4 +76,11 @@
         </geometry>
       </visual>
+      <xacro:unless value="${use_cylinder_collision_model}">
+        <collision>
+          <geometry>
+            <mesh filename="package://franka_description/meshes/collision/finger.stl"/>
+          </geometry>
+        </collision>
+      </xacro:unless>
       <!-- for simulation -->
       <inertial>
@@ -81,7 +98,15 @@
         </geometry>
       </visual>
+      <xacro:unless value="${use_cylinder_collision_model}">
+        <collision>
+          <origin xyz="0 0 0" rpy="0 0 ${pi}"/>
+          <geometry>
+            <mesh filename="package://franka_description/meshes/collision/finger.stl"/>
+          </geometry>
+        </collision>
+      </xacro:unless>
       <!-- for simulation -->
       <inertial>
-        <origin xyz="0 0 0" rpy="0 0 0" />
+        <origin xyz="0 0 0" rpy="0 0 ${pi}" />
         <mass value="0.01" />
         <inertia ixx="0.1" ixy="0.0" ixz="0.0" iyy="0.1" iyz="0.0" izz="0.1" />

File: franka_description/robots/panda_arm.urdf.xacro (robot description, xacro)
@@ -2,4 +2,5 @@
 <robot xmlns:xacro="http://www.ros.org/wiki/xacro" name="panda">
   <xacro:arg name="arm_id" default="panda"/>
+  <xacro:arg name="use_cylinder_collision_model" default="true"/>
   <xacro:include filename="$(find franka_description)/robots/panda_arm.xacro" />
   <!-- for simulation -->
@@ -7,5 +8,7 @@
   <xacro:include filename="$(find franka_description)/robots/panda.control.xacro"/>
   <!-- end for simulation -->
-  <xacro:panda_arm xyz="0 0 0" rpy="0 0 0" connected_to="world" arm_id="$(arg arm_id)" safety_distance="0.03"/>
+  <link name="world"/>
+  <xacro:panda_arm xyz="0 0 0" rpy="0 0 0" connected_to="world" arm_id="$(arg arm_id)"
+    safety_distance="0.03" use_cylinder_collision_model="$(arg use_cylinder_collision_model)"/>
   <!-- for simulation -->
   <xacro:arm_gazebo arm_id="$(arg arm_id)"/>

File: franka_description/robots/panda_arm.xacro (robot description, xacro)
@@ -3,5 +3,6 @@
   <!-- safety_distance: Minimum safety distance in [m] by which the collision volumes are expanded and which is enforced during robot motions -->
   <!-- arm_id: Namespace of the panda arm. Serves to differentiate between arms in case of multiple instances. -->
-  <xacro:macro name="panda_arm" params="arm_id:='panda' description_pkg:='franka_description' connected_to:='' xyz:='0 0 0' rpy:='0 0 0' safety_distance:=0">
+  <xacro:macro name="panda_arm" params="arm_id:='panda' description_pkg:='franka_description'
+    connected_to:='' xyz:='0 0 0' rpy:='0 0 0' safety_distance:=0 use_cylinder_collision_model:='true'">
     <xacro:unless value="${not connected_to}">
       <joint name="virtual_joint" type="fixed">
@@ -14,5 +15,6 @@
       </joint>
     </xacro:unless>
-    <xacro:macro name="arm_link" params="name visual_mesh:='' collision_mesh:='' mass:='0.0' **cylinder_collision_model">
+    <xacro:macro name="arm_link" params="name visual_mesh:='' collision_mesh:='' mass:='0.0'
+      **cylinder_collision_model use_cylinder_collision_model:='true'">
       <link name="${name}">
         <xacro:unless value="${not visual_mesh}">
@@ -23,15 +25,16 @@
           </visual>
         </xacro:unless>
-        <xacro:unless value="${not collision_mesh}">
-          <collision>
-            <geometry>
-              <mesh filename="${collision_mesh}"/>
-            </geometry>
-          </collision>
-        </xacro:unless>
-        <!-- Fallback to cylinder-collision model if no mesh is specified-->
-        <xacro:if value="${not collision_mesh}">
+        <xacro:if value="${use_cylinder_collision_model}">
           <xacro:insert_block name="cylinder_collision_model"/>
         </xacro:if>
+        <!-- Fallback to mesh model, when cylinder collision model is requested to be not used and
+             there is a specified collision mesh.-->
+        <xacro:unless value="${use_cylinder_collision_model and (not collision_mesh)}">
+          <collision>
+            <geometry>
+              <mesh filename="${collision_mesh}"/>
+            </geometry>
+          </collision>
+        </xacro:unless>
         <!-- for simulation -->
         <inertial>
@@ -63,228 +66,268 @@
       </joint>
     </xacro:macro>
-    <xacro:arm_link name="${arm_id}_link0" visual_mesh="package://${description_pkg}/meshes/visual/link0.dae"
-      collision_mesh="package://${description_pkg}/meshes/collision/link0.stl" mass="3.06">
-      <cylinder_collision_model>
-        <collision>
-          <origin xyz="0 0 -0.1915" rpy="0 0 0"/>
-          <geometry>
-            <cylinder radius="${0.06+safety_distance}" length="0.2830" />
-          </geometry>
-        </collision>
-        <collision>
-          <origin xyz="0 0 -0.333" rpy="0 0 0"/>
-          <geometry>
-            <sphere radius="${0.06+safety_distance}" />
-          </geometry>
-        </collision>
-        <collision>
-          <origin xyz="0 0 -0.05" rpy="0 0 0"/>
-          <geometry>
-            <sphere radius="${0.06+safety_distance}" />
-          </geometry>
-        </collision>
-      </cylinder_collision_model>
-    </xacro:arm_link>
-    <xacro:arm_link name="${arm_id}_link1" visual_mesh="package://${description_pkg}/meshes/visual/link1.dae"
-      collision_mesh="package://${description_pkg}/meshes/collision/link1.stl" mass="2.34">
-      <cylinder_collision_model>
-        <collision>
-          <origin xyz="0 0 -0.1915" rpy="0 0 0"/>
-          <geometry>
-            <cylinder radius="${0.06+safety_distance}" length="0.2830" />
-          </geometry>
-        </collision>
-        <collision>
-          <origin xyz="0 0 -0.333" rpy="0 0 0"/>
-          <geometry>
-            <sphere radius="${0.06+safety_distance}" />
-          </geometry>
-        </collision>
-        <collision>
-          <origin xyz="0 0 -0.05" rpy="0 0 0"/>
-          <geometry>
-            <sphere radius="${0.06+safety_distance}" />
-          </geometry>
-        </collision>
-      </cylinder_collision_model>
-    </xacro:arm_link>
-    <xacro:arm_link name="${arm_id}_link2" visual_mesh="package://${description_pkg}/meshes/visual/link2.dae"
-      collision_mesh="package://${description_pkg}/meshes/collision/link2.stl" mass="2.36">
-      <cylinder_collision_model>
-        <collision>
-          <origin xyz="0 0 0" rpy="0 0 0"/>
-          <geometry>
-            <cylinder radius="${0.06+safety_distance}" length="0.12" />
-          </geometry>
-        </collision>
-        <collision>
-          <origin xyz="0 0 -0.06" rpy="0 0 0"/>
-          <geometry>
-            <sphere radius="${0.06+safety_distance}" />
-          </geometry>
-        </collision>
-        <collision>
-          <origin xyz="0 0 0.06" rpy="0 0 0"/>
-          <geometry>
-            <sphere radius="${0.06+safety_distance}" />
-          </geometry>
-        </collision>
-      </cylinder_collision_model>
-    </xacro:arm_link>
-    <xacro:arm_link name="${arm_id}_link3" visual_mesh="package://${description_pkg}/meshes/visual/link3.dae"
-      collision_mesh="package://${description_pkg}/meshes/collision/link3.stl" mass="2.38">
-      <cylinder_collision_model>
-        <collision>
-          <origin xyz="0 0 -0.145" rpy="0 0 0"/>
-          <geometry>
-            <cylinder radius="${0.06+safety_distance}" length="0.15" />
-          </geometry>
-        </collision>
-        <collision>
-          <origin xyz="0 0 -0.22" rpy="0 0 0"/>
-          <geometry>
-            <sphere radius="${0.06+safety_distance}" />
-          </geometry>
-        </collision>
-        <collision>
-          <origin xyz="0 0 -0.07" rpy="0 0 0"/>
-          <geometry>
-            <sphere radius="${0.06+safety_distance}" />
-          </geometry>
-        </collision>
-      </cylinder_collision_model>
-    </xacro:arm_link>
-    <xacro:arm_link name="${arm_id}_link4" visual_mesh="package://${description_pkg}/meshes/visual/link4.dae"
-      collision_mesh="package://${description_pkg}/meshes/collision/link4.stl" mass="2.43">
-      <cylinder_collision_model>
-        <collision>
-          <origin xyz="0 0 0" rpy="0 0 0"/>
-          <geometry>
-            <cylinder radius="${0.06+safety_distance}" length="0.12" />
-          </geometry>
-        </collision>
-        <collision>
-          <origin xyz="0 0 0.06" rpy="0 0 0"/>
-          <geometry>
-            <sphere radius="${0.06+safety_distance}" />
-          </geometry>
-        </collision>
-        <collision>
-          <origin xyz="0 0 -0.06" rpy="0 0 0"/>
-          <geometry>
-            <sphere radius="${0.06+safety_distance}" />
-          </geometry>
-        </collision>
-      </cylinder_collision_model>
-    </xacro:arm_link>
-    <xacro:arm_link name="${arm_id}_link5" visual_mesh="package://${description_pkg}/meshes/visual/link5.dae"
-      collision_mesh="package://${description_pkg}/meshes/collision/link5.stl" mass="3.5">
-      <cylinder_collision_model>
-        <collision>
-          <origin xyz="0 0 -0.26" rpy="0 0 0"/>
-          <geometry>
-            <cylinder radius="${0.06+safety_distance}" length="0.1" />
-          </geometry>
-        </collision>
-        <collision>
-          <origin xyz="0 0 -0.31" rpy="0 0 0"/>
-          <geometry>
-            <sphere radius="${0.06+safety_distance}" />
-          </geometry>
-        </collision>
-        <collision>
-          <origin xyz="0 0 -0.21" rpy="0 0 0"/>
-          <geometry>
-            <sphere radius="${0.06+safety_distance}" />
-          </geometry>
-        </collision>
-        <collision>
-          <origin xyz="0 0.08 -0.13" rpy="0 0 0"/>
-          <geometry>
-            <cylinder radius="${0.025+safety_distance}" length="0.14" />
-          </geometry>
-        </collision>
-        <collision>
-          <origin xyz="0 0.08 -0.06" rpy="0 0 0"/>
-          <geometry>
-            <sphere radius="${0.025+safety_distance}" />
-          </geometry>
-        </collision>
-        <collision>
-          <origin xyz="0 0.08 -0.20" rpy="0 0 0"/>
-          <geometry>
-            <sphere radius="${0.025+safety_distance}" />
-          </geometry>
-        </collision>
-      </cylinder_collision_model>
-    </xacro:arm_link>
-    <xacro:arm_link name="${arm_id}_link6" visual_mesh="package://${description_pkg}/meshes/visual/link6.dae"
-      collision_mesh="package://${description_pkg}/meshes/collision/link6.stl" mass="1.47">
-      <cylinder_collision_model>
-        <collision>
-          <origin xyz="0 0 -0.03" rpy="0 0 0"/>
-          <geometry>
-            <cylinder radius="${0.05+safety_distance}" length="0.08" />
-          </geometry>
-        </collision>
-        <collision>
-          <origin xyz="0 0 0.01" rpy="0 0 0"/>
-          <geometry>
-            <sphere radius="${0.05+safety_distance}" />
-          </geometry>
-        </collision>
-        <collision>
-          <origin xyz="0 0 -0.07" rpy="0 0 0"/>
-          <geometry>
-            <sphere radius="${0.05+safety_distance}" />
-          </geometry>
-        </collision>
-      </cylinder_collision_model>
-    </xacro:arm_link>
-    <xacro:arm_link name="${arm_id}_link7" visual_mesh="package://${description_pkg}/meshes/visual/link7.dae"
-      collision_mesh="package://${description_pkg}/meshes/collision/link7.stl" mass="0.45">
-      <cylinder_collision_model>
-        <collision>
-          <origin xyz="0 0 0.01" rpy="0 0 0"/>
-          <geometry>
-            <cylinder radius="${0.04+safety_distance}" length="0.14" />
-          </geometry>
-        </collision>
-        <collision>
-          <origin xyz="0 0 0.08" rpy="0 0 0"/>
-          <geometry>
-            <sphere radius="${0.04+safety_distance}"  />
-          </geometry>
-        </collision>
-        <collision>
-          <origin xyz="0 0 -0.06" rpy="0 0 0"/>
-          <geometry>
-            <sphere radius="${0.04+safety_distance}"  />
-          </geometry>
-        </collision>
-      </cylinder_collision_model>
-    </xacro:arm_link>
-    <xacro:arm_link name="${arm_id}_link8">
-      <cylinder_collision_model>
-        <collision>
-          <origin xyz="0.0424 0.0424 -0.0250" rpy="${pi} ${pi/2} ${pi/2}"/>
-          <geometry>
-            <cylinder radius="${0.03+safety_distance}"  length="0.01" />
-          </geometry>
-        </collision>
-        <collision>
-          <origin xyz="0.0424 0.0424 -0.02" rpy="0 0 0"/>
-          <geometry>
-            <sphere radius="${0.03+safety_distance}"  />
-          </geometry>
-        </collision>
-        <collision>
-          <origin xyz="0.0424 0.0424 -0.03" rpy="0 0 0"/>
-          <geometry>
-            <sphere radius="${0.03+safety_distance}"  />
-          </geometry>
-        </collision>
-      </cylinder_collision_model>
-    </xacro:arm_link>
+    <xacro:if value="${use_cylinder_collision_model}">
+      <xacro:arm_link name="${arm_id}_link0" visual_mesh="package://${description_pkg}/meshes/visual/link0.dae" mass="3.06">
+        <cylinder_collision_model>
+          <collision>
+            <origin xyz="0 0 -0.1915" rpy="0 0 0"/>
+            <geometry>
+              <cylinder radius="${0.06+safety_distance}" length="0.2830" />
+            </geometry>
+          </collision>
+          <collision>
+            <origin xyz="0 0 -0.333" rpy="0 0 0"/>
+            <geometry>
+              <sphere radius="${0.06+safety_distance}" />
+            </geometry>
+          </collision>
+          <collision>
+            <origin xyz="0 0 -0.05" rpy="0 0 0"/>
+            <geometry>
+              <sphere radius="${0.06+safety_distance}" />
+            </geometry>
+          </collision>
+        </cylinder_collision_model>
+      </xacro:arm_link>
+      <xacro:arm_link name="${arm_id}_link1" visual_mesh="package://${description_pkg}/meshes/visual/link1.dae" mass="2.34">
+        <cylinder_collision_model>
+          <collision>
+            <origin xyz="0 0 -0.1915" rpy="0 0 0"/>
+            <geometry>
+              <cylinder radius="${0.06+safety_distance}" length="0.2830" />
+            </geometry>
+          </collision>
+          <collision>
+            <origin xyz="0 0 -0.333" rpy="0 0 0"/>
+            <geometry>
+              <sphere radius="${0.06+safety_distance}" />
+            </geometry>
+          </collision>
+          <collision>
+            <origin xyz="0 0 -0.05" rpy="0 0 0"/>
+            <geometry>
+              <sphere radius="${0.06+safety_distance}" />
+            </geometry>
+          </collision>
+        </cylinder_collision_model>
+      </xacro:arm_link>
+      <xacro:arm_link name="${arm_id}_link2" visual_mesh="package://${description_pkg}/meshes/visual/link2.dae" mass="2.36">
+        <cylinder_collision_model>
+          <collision>
+            <origin xyz="0 0 0" rpy="0 0 0"/>
+            <geometry>
+              <cylinder radius="${0.06+safety_distance}" length="0.12" />
+            </geometry>
+          </collision>
+          <collision>
+            <origin xyz="0 0 -0.06" rpy="0 0 0"/>
+            <geometry>
+              <sphere radius="${0.06+safety_distance}" />
+            </geometry>
+          </collision>
+          <collision>
+            <origin xyz="0 0 0.06" rpy="0 0 0"/>
+            <geometry>
+              <sphere radius="${0.06+safety_distance}" />
+            </geometry>
+          </collision>
+        </cylinder_collision_model>
+      </xacro:arm_link>
+      <xacro:arm_link name="${arm_id}_link3" visual_mesh="package://${description_pkg}/meshes/visual/link3.dae" mass="2.38">
+        <cylinder_collision_model>
+          <collision>
+            <origin xyz="0 0 -0.145" rpy="0 0 0"/>
+            <geometry>
+              <cylinder radius="${0.06+safety_distance}" length="0.15" />
+            </geometry>
+          </collision>
+          <collision>
+            <origin xyz="0 0 -0.22" rpy="0 0 0"/>
+            <geometry>
+              <sphere radius="${0.06+safety_distance}" />
+            </geometry>
+          </collision>
+          <collision>
+            <origin xyz="0 0 -0.07" rpy="0 0 0"/>
+            <geometry>
+              <sphere radius="${0.06+safety_distance}" />
+            </geometry>
+          </collision>
+        </cylinder_collision_model>
+      </xacro:arm_link>
+      <xacro:arm_link name="${arm_id}_link4" visual_mesh="package://${description_pkg}/meshes/visual/link4.dae" mass="2.43">
+        <cylinder_collision_model>
+          <collision>
+            <origin xyz="0 0 0" rpy="0 0 0"/>
+            <geometry>
+              <cylinder radius="${0.06+safety_distance}" length="0.12" />
+            </geometry>
+          </collision>
+          <collision>
+            <origin xyz="0 0 0.06" rpy="0 0 0"/>
+            <geometry>
+              <sphere radius="${0.06+safety_distance}" />
+            </geometry>
+          </collision>
+          <collision>
+            <origin xyz="0 0 -0.06" rpy="0 0 0"/>
+            <geometry>
+              <sphere radius="${0.06+safety_distance}" />
+            </geometry>
+          </collision>
+        </cylinder_collision_model>
+      </xacro:arm_link>
+      <xacro:arm_link name="${arm_id}_link5" visual_mesh="package://${description_pkg}/meshes/visual/link5.dae" mass="3.5">
+        <cylinder_collision_model>
+          <collision>
+            <origin xyz="0 0 -0.26" rpy="0 0 0"/>
+            <geometry>
+              <cylinder radius="${0.06+safety_distance}" length="0.1" />
+            </geometry>
+          </collision>
+          <collision>
+            <origin xyz="0 0 -0.31" rpy="0 0 0"/>
+            <geometry>
+              <sphere radius="${0.06+safety_distance}" />
+            </geometry>
+          </collision>
+          <collision>
+            <origin xyz="0 0 -0.21" rpy="0 0 0"/>
+            <geometry>
+              <sphere radius="${0.06+safety_distance}" />
+            </geometry>
+          </collision>
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