Commit message: If-guard Gazebo-specific stuff for to reduce parameter footprint in real usage.

File: franka_description/robots/hand.urdf.xacro (robot description, xacro)
@@ -2,14 +2,15 @@
 <robot xmlns:xacro="http://www.ros.org/wiki/xacro" name="hand">
   <xacro:arg name="use_cylinder_collision_model" default="true"/>
+  <xacro:arg name="use_gazebo_sim" default="false"/>
   <xacro:include filename="hand.xacro"/>
-  <!-- for simulation -->
-  <xacro:include filename="$(find franka_description)/robots/panda.gazebo.xacro"/>
-  <xacro:include filename="$(find franka_description)/robots/panda.control.xacro"/>
-  <!-- end for simulation -->
+  <xacro:if value="$(arg use_gazebo_sim)">
+    <xacro:include filename="$(find franka_description)/robots/panda.gazebo.xacro"/>
+    <xacro:include filename="$(find franka_description)/robots/panda.control.xacro"/>
+  </xacro:if>
   <xacro:hand ns="panda" rpy="0 0 ${-pi/4}" connected_to="panda_link8" safety_distance="0.03"
     use_cylinder_collision_model="$(arg use_cylinder_collision_model)"/>
-  <!-- for simulation -->
-  <xacro:hand_gazebo arm_id="$(arg arm_id)"/>
-  <xacro:hand_control arm_id="$(arg arm_id)"/>
-  <!-- end for simulation -->
+  <xacro:if value="$(arg use_gazebo_sim)">
+    <xacro:hand_gazebo arm_id="$(arg arm_id)"/>
+    <xacro:hand_control arm_id="$(arg arm_id)"/>
+  </xacro:if>
 </robot>

File: franka_description/robots/hand.xacro (robot description, xacro)
@@ -1,4 +1,5 @@
 <?xml version="1.0" encoding="utf-8"?>
 <robot xmlns:xacro="http://www.ros.org/wiki/xacro" name="hand">
+  <xacro:arg name="use_gazebo_sim" default="false"/>
   <!-- safety_distance: Minimum safety distance in [m] by which the collision volumes are expanded and which is enforced during robot motions -->
   <xacro:macro name="hand" params="connected_to:='' ns:='' rpy:='0 0 0' xyz:='0 0 0' safety_distance:=0
@@ -62,11 +63,11 @@
         </collision>
       </xacro:unless>
-      <!-- for simulation -->
-      <inertial>
-        <origin xyz="0 0 0" rpy="0 0 0" />
-        <mass value="0.68" />
-        <inertia ixx="0.1" ixy="0.0" ixz="0.0" iyy="0.1" iyz="0.0" izz="0.1" />
-      </inertial>
-      <!-- end for simulation -->
+      <xacro:if value="$(arg use_gazebo_sim)">
+        <inertial>
+          <origin xyz="0 0 0" rpy="0 0 0" />
+          <mass value="0.68" />
+          <inertia ixx="0.1" ixy="0.0" ixz="0.0" iyy="0.1" iyz="0.0" izz="0.1" />
+        </inertial>
+      </xacro:if>
     </link>
     <link name="${ns}_leftfinger">
@@ -83,11 +84,11 @@
         </collision>
       </xacro:unless>
-      <!-- for simulation -->
-      <inertial>
-        <origin xyz="0 0 0" rpy="0 0 0" />
-        <mass value="0.01" />
-        <inertia ixx="0.1" ixy="0.0" ixz="0.0" iyy="0.1" iyz="0.0" izz="0.1" />
-      </inertial>
-      <!-- end for simulation -->
+      <xacro:if value="$(arg use_gazebo_sim)">
+        <inertial>
+          <origin xyz="0 0 0" rpy="0 0 0" />
+          <mass value="0.01" />
+          <inertia ixx="0.1" ixy="0.0" ixz="0.0" iyy="0.1" iyz="0.0" izz="0.1" />
+        </inertial>
+      </xacro:if>
     </link>
     <link name="${ns}_rightfinger">
@@ -106,11 +107,11 @@
         </collision>
       </xacro:unless>
-      <!-- for simulation -->
-      <inertial>
-        <origin xyz="0 0 0" rpy="0 0 ${pi}" />
-        <mass value="0.01" />
-        <inertia ixx="0.1" ixy="0.0" ixz="0.0" iyy="0.1" iyz="0.0" izz="0.1" />
-      </inertial>
-      <!-- end for simulation -->
+      <xacro:if value="$(arg use_gazebo_sim)">
+        <inertial>
+          <origin xyz="0 0 0" rpy="0 0 ${pi}" />
+          <mass value="0.01" />
+          <inertia ixx="0.1" ixy="0.0" ixz="0.0" iyy="0.1" iyz="0.0" izz="0.1" />
+        </inertial>
+      </xacro:if>
    </link>
     <joint name="${ns}_finger_joint1" type="prismatic">
@@ -127,5 +128,7 @@
       <axis xyz="0 -1 0"/>
       <limit effort="20" lower="0.0" upper="0.04" velocity="0.2"/>
-      <mimic joint="${ns}_finger_joint1" />
+      <xacro:unless value="$(arg use_gazebo_sim)">
+        <mimic joint="${ns}_finger_joint1" />
+      </xacro:unless>
     </joint>
   </xacro:macro>

File: franka_description/robots/panda.control.xacro (robot description, xacro)
@@ -26,6 +26,3 @@
         <xacro:joint_control transmission="${arm_id}_rightfinger" joint="${arm_id}_finger_joint2" motor="${arm_id}_finger_joint2"/>
     </xacro:macro>
-    <gazebo>
-        <plugin name="gazebo_ros_control" filename="libgazebo_ros_control.so"/>
-    </gazebo>
 </robot>

File: franka_description/robots/panda_arm.urdf.xacro (robot description, xacro)
@@ -3,15 +3,19 @@
   <xacro:arg name="arm_id" default="panda"/>
   <xacro:arg name="use_cylinder_collision_model" default="true"/>
+  <xacro:arg name="use_gazebo_sim" default="false"/>
   <xacro:include filename="$(find franka_description)/robots/panda_arm.xacro" />
-  <!-- for simulation -->
-  <xacro:include filename="$(find franka_description)/robots/panda.gazebo.xacro"/>
-  <xacro:include filename="$(find franka_description)/robots/panda.control.xacro"/>
-  <!-- end for simulation -->
+  <xacro:if value="$(arg use_gazebo_sim)">
+    <xacro:include filename="$(find franka_description)/robots/panda.gazebo.xacro"/>
+    <xacro:include filename="$(find franka_description)/robots/panda.control.xacro"/>
+  </xacro:if>
   <link name="world"/>
   <xacro:panda_arm xyz="0 0 0" rpy="0 0 0" connected_to="world" arm_id="$(arg arm_id)"
     safety_distance="0.03" use_cylinder_collision_model="$(arg use_cylinder_collision_model)"/>
-  <!-- for simulation -->
-  <xacro:arm_gazebo arm_id="$(arg arm_id)"/>
-  <xacro:arm_control arm_id="$(arg arm_id)"/>
-  <!-- end for simulation -->
+  <xacro:if value="$(arg use_gazebo_sim)">
+    <xacro:arm_gazebo arm_id="$(arg arm_id)"/>
+    <xacro:arm_control arm_id="$(arg arm_id)"/>
+    <gazebo>
+        <plugin name="gazebo_ros_control" filename="libgazebo_ros_control.so"/>
+    </gazebo>
+  </xacro:if>
 </robot>

File: franka_description/robots/panda_arm.xacro (robot description, xacro)
@@ -1,4 +1,5 @@
 <?xml version='1.0' encoding='utf-8'?>
 <robot xmlns:xacro="http://www.ros.org/wiki/xacro" name="panda">
+  <xacro:arg name="use_gazebo_sim" default="false"/>
   <!-- safety_distance: Minimum safety distance in [m] by which the collision volumes are expanded and which is enforced during robot motions -->
   <!-- arm_id: Namespace of the panda arm. Serves to differentiate between arms in case of multiple instances. -->
@@ -10,7 +11,7 @@
         <child link="${arm_id}_link0"/>
         <origin rpy="${rpy}" xyz="${xyz}"/>
-        <!-- for simulation -->
-        <dynamics damping="1.0"/>
-        <!-- end for simulation -->
+        <xacro:if value="$(arg use_gazebo_sim)">
+          <dynamics damping="1.0"/>
+        </xacro:if>
       </joint>
     </xacro:unless>
@@ -37,11 +38,11 @@
           </collision>
         </xacro:unless>
-        <!-- for simulation -->
-        <inertial>
-          <origin xyz="0 0 0" rpy="0 0 0" />
-          <mass value="${mass}"/>
-          <inertia ixx="0.3" ixy="0.0" ixz="0.0" iyy="0.3" iyz="0.0" izz="0.3" />
-        </inertial>
-        <!-- end for simulation -->
+        <xacro:if value="$(arg use_gazebo_sim)">
+          <inertial>
+            <origin xyz="0 0 0" rpy="0 0 0" />
+            <mass value="${mass}"/>
+            <inertia ixx="0.3" ixy="0.0" ixz="0.0" iyy="0.3" iyz="0.0" izz="0.3" />
+          </inertial>
+        </xacro:if>
       </link>
     </xacro:macro>
