Commit message: Update and improve usage

File: franka_description/robots/panda.gazebo.xacro (robot description, xacro)
@@ -1,77 +1,31 @@
-<?xml version="1.0"?>
+<?xml version='1.0' encoding='utf-8'?>
 <robot xmlns:xacro="http://www.ros.org/wiki/xacro">
-    <xacro:macro name="panda_gazebo" params="robot_name">
-        <!-- Link0 -->
-        <gazebo reference="${robot_name}_link0">
-            <material>Gazebo/Grey</material>
-            <mu1>0.2</mu1>
-            <mu2>0.2</mu2>
-        </gazebo>
-        <!-- Link1 -->
-        <gazebo reference="${robot_name}_link1">
-            <material>Gazebo/White</material>
-            <mu1>0.2</mu1>
-            <mu2>0.2</mu2>
-        </gazebo>
-        <!-- Link2 -->
-        <gazebo reference="${robot_name}_link2">
-            <material>Gazebo/White</material>
-            <mu1>0.2</mu1>
-            <mu2>0.2</mu2>
-        </gazebo>
-        <!-- Link3 -->
-        <gazebo reference="${robot_name}_link3">
-            <material>Gazebo/White</material>
-            <mu1>0.2</mu1>
-            <mu2>0.2</mu2>
-        </gazebo>
-        <!-- Link4 -->
-        <gazebo reference="${robot_name}_link4">
-            <material>Gazebo/White</material>
-            <mu1>0.2</mu1>
-            <mu2>0.2</mu2>
-        </gazebo>
-        <!-- Link5 -->
-        <gazebo reference="${robot_name}_link5">
-            <material>Gazebo/White</material>
-            <mu1>0.2</mu1>
-            <mu2>0.2</mu2>
-        </gazebo>
-        <!-- Link6 -->
-        <gazebo reference="${robot_name}_link6">
-            <material>Gazebo/White</material>
-            <mu1>0.2</mu1>
-            <mu2>0.2</mu2>
-        </gazebo>
-        <!-- Link7 -->
-        <gazebo reference="${robot_name}_link7">
-            <material>Gazebo/Grey</material>
-            <mu1>0.2</mu1>
-            <mu2>0.2</mu2>
-        </gazebo>
-        <!-- Link8 -->
-        <gazebo reference="${robot_name}_link8">
-            <material>Gazebo/Grey</material>
-            <mu1>0.2</mu1>
-            <mu2>0.2</mu2>
-        </gazebo>
-        <!-- LinkHand -->
-        <gazebo reference="${robot_name}_hand">
-            <material>Gazebo/Grey</material>
-            <mu1>0.2</mu1>
-            <mu2>0.2</mu2>
-        </gazebo>
-        <!-- LinkRightFinger -->
-        <gazebo reference="${robot_name}_rightfinger">
-            <material>Gazebo/Grey</material>
-            <mu1>0.2</mu1>
-            <mu2>0.2</mu2>
-        </gazebo>
-        <!-- LinkLeftFinger -->
-        <gazebo reference="${robot_name}_leftfinger">
-            <material>Gazebo/Grey</material>
-            <mu1>0.2</mu1>
-            <mu2>0.2</mu2>
-        </gazebo>
+    <xacro:macro name="panda_gazebo" params="arm_id">
+        <xacro:macro name="arm_gazebo" params="link">
+            <gazebo reference="${link}">
+                <material>Gazebo/White</material>
+                <mu1>0.2</mu1>
+                <mu2>0.2</mu2>
+            </gazebo>
+        </xacro:macro>
+        <xacro:macro name="hand_gazebo" params="link">
+            <gazebo reference="${link}">
+                <material>Gazebo/Grey</material>
+                <mu1>0.2</mu1>
+                <mu2>0.2</mu2>
+            </gazebo>
+        </xacro:macro>
+        <xacro:arm_gazebo link="${arm_id}_link0"/>
+        <xacro:arm_gazebo link="${arm_id}_link1"/>
+        <xacro:arm_gazebo link="${arm_id}_link2"/>
+        <xacro:arm_gazebo link="${arm_id}_link3"/>
+        <xacro:arm_gazebo link="${arm_id}_link4"/>
+        <xacro:arm_gazebo link="${arm_id}_link5"/>
+        <xacro:arm_gazebo link="${arm_id}_link6"/>
+        <xacro:hand_gazebo link="${arm_id}_link7"/>
+        <xacro:hand_gazebo link="${arm_id}_link8"/>
+        <xacro:hand_gazebo link="${arm_id}_hand"/>
+        <xacro:hand_gazebo link="${arm_id}_rightfinger"/>
+        <xacro:hand_gazebo link="${arm_id}_leftfinger"/>
     </xacro:macro>
 </robot>

File: franka_description/robots/panda_arm.xacro (robot description, xacro)
@@ -4,20 +4,13 @@
   <!-- arm_id: Namespace of the panda arm. Serves to differentiate between arms in case of multiple instances. -->
   <xacro:macro name="panda_arm" params="arm_id:='panda' description_pkg:='franka_description' connected_to:='' xyz:='0 0 0' rpy:='0 0 0' safety_distance:=0">
+    <link name="world" />
     <xacro:unless value="${not connected_to}">
-      <joint name="${arm_id}_joint_${connected_to}" type="fixed">
+      <joint name="virtual_joint" type="fixed">
         <parent link="${connected_to}"/>
         <child link="${arm_id}_link0"/>
         <origin rpy="${rpy}" xyz="${xyz}"/>
+        <dynamics damping="1.0"/>
       </joint>
     </xacro:unless>
-    <!-- for simulation -->
-    <link name="world" />
-    <joint name="robot_to_world" type="fixed">
-      <parent link="world" />
-      <child link="${arm_id}_link0" />
-      <origin xyz="0.0 0.0 0.0" rpy="0.0 0.0 0.0" />
-    </joint>
-    <xacro:property name="joint_damping" value="1.0"/>
-    <!-- end for simulation -->
     <link name="${arm_id}_link0">
       <visual>
@@ -92,5 +85,5 @@
       <limit effort="87" lower="-2.8973" upper="2.8973" velocity="2.1750"/>
       <!-- for simulation -->
-      <dynamics damping="${joint_damping}"/>
+      <dynamics damping="1.0"/>
       <!-- end for simulation -->
     </joint>
@@ -135,5 +128,5 @@
       <limit effort="87" lower="-1.7628" upper="1.7628" velocity="2.1750"/>
       <!-- for simulation -->
-      <dynamics damping="${joint_damping}"/>
+      <dynamics damping="1.0"/>
       <!-- end for simulation -->
     </joint>
@@ -178,5 +171,5 @@
       <limit effort="87" lower="-2.8973" upper="2.8973" velocity="2.1750"/>
       <!-- for simulation -->
-      <dynamics damping="${joint_damping}"/>
+      <dynamics damping="1.0"/>
       <!-- end for simulation -->
     </joint>
@@ -221,5 +214,5 @@
       <limit effort="87" lower="-3.0718" upper="-0.0698" velocity="2.1750"/>
       <!-- for simulation -->
-      <dynamics damping="${joint_damping}"/>
+      <dynamics damping="1.0"/>
       <!-- end for simulation -->
     </joint>
@@ -282,5 +275,5 @@
       <limit effort="12" lower="-2.8973" upper="2.8973" velocity="2.6100"/>
       <!-- for simulation -->
-      <dynamics damping="${joint_damping}"/>
+      <dynamics damping="1.0"/>
       <!-- end for simulation -->
     </joint>
@@ -325,5 +318,5 @@
       <limit effort="12" lower="-0.0175" upper="3.7525" velocity="2.6100"/>
       <!-- for simulation -->
-      <dynamics damping="${joint_damping}"/>
+      <dynamics damping="1.0"/>
       <!-- end for simulation -->
     </joint>
@@ -368,5 +361,5 @@
       <limit effort="12" lower="-2.8973" upper="2.8973" velocity="2.6100"/>
       <!-- for simulation -->
-      <dynamics damping="${joint_damping}"/>
+      <dynamics damping="1.0"/>
       <!-- end for simulation -->
     </joint>

File: franka_description/robots/panda_arm_hand.urdf.xacro (robot description, xacro)
@@ -6,12 +6,11 @@
   <!-- for simulation -->
   <xacro:include filename="$(find franka_description)/robots/panda.gazebo.xacro"/>
-  <xacro:include filename="panda.transmission.xacro"/>
+  <xacro:include filename="$(find franka_description)/robots/panda.control.xacro"/>
   <!-- end for simulation -->
-  <xacro:panda_arm />
+  <xacro:panda_arm xyz="0 0 0" rpy="0 0 0" connected_to="world" arm_id="panda"/>
   <xacro:hand ns="panda" rpy="0 0 ${-pi/4}" connected_to="panda_link8" safety_distance="0.03"/>
   <!-- for simulation -->
-  <xacro:arg name="robot_name" default="panda"/>
-  <xacro:panda_gazebo robot_name="$(arg robot_name)" />
-  <xacro:panda_transmission robot_name="$(arg robot_name)" load_hand="true" />
+  <xacro:panda_gazebo arm_id="panda"/>
+  <xacro:panda_control arm_id="panda" load_hand="true" />
   <!-- end for simulation -->
 </robot>

Commit message: Rename material macro.

File: franka_description/robots/panda.gazebo.xacro (robot description, xacro)
@@ -2,5 +2,5 @@
 <robot xmlns:xacro="http://www.ros.org/wiki/xacro">
     <xacro:macro name="arm_gazebo" params="arm_id">
-        <xacro:macro name="arm_link_gazebo" params="link">
+        <xacro:macro name="arm_material" params="link">
             <gazebo reference="${link}">
                 <material>Gazebo/White</material>
@@ -9,16 +9,16 @@
             </gazebo>
         </xacro:macro>
-        <xacro:arm_link_gazebo link="${arm_id}_link0"/>
-        <xacro:arm_link_gazebo link="${arm_id}_link1"/>
-        <xacro:arm_link_gazebo link="${arm_id}_link2"/>
-        <xacro:arm_link_gazebo link="${arm_id}_link3"/>
-        <xacro:arm_link_gazebo link="${arm_id}_link4"/>
-        <xacro:arm_link_gazebo link="${arm_id}_link5"/>
-        <xacro:arm_link_gazebo link="${arm_id}_link6"/>
-        <xacro:arm_link_gazebo link="${arm_id}_link7"/>
-        <xacro:arm_link_gazebo link="${arm_id}_link8"/>
+        <xacro:arm_material link="${arm_id}_link0"/>
+        <xacro:arm_material link="${arm_id}_link1"/>
+        <xacro:arm_material link="${arm_id}_link2"/>
+        <xacro:arm_material link="${arm_id}_link3"/>
+        <xacro:arm_material link="${arm_id}_link4"/>
+        <xacro:arm_material link="${arm_id}_link5"/>
+        <xacro:arm_material link="${arm_id}_link6"/>
+        <xacro:arm_material link="${arm_id}_link7"/>
+        <xacro:arm_material link="${arm_id}_link8"/>
     </xacro:macro>
     <xacro:macro name="hand_gazebo" params="arm_id">
-        <xacro:macro name="hand_link_gazebo" params="link">
+        <xacro:macro name="hand_material" params="link">
             <gazebo reference="${link}">
                 <material>Gazebo/Grey</material>
@@ -27,7 +27,7 @@
             </gazebo>
         </xacro:macro>
-        <xacro:hand_link_gazebo link="${arm_id}_hand"/>
-        <xacro:hand_link_gazebo link="${arm_id}_rightfinger"/>
-        <xacro:hand_link_gazebo link="${arm_id}_leftfinger"/>
+        <xacro:hand_material link="${arm_id}_hand"/>
+        <xacro:hand_material link="${arm_id}_rightfinger"/>
+        <xacro:hand_material link="${arm_id}_leftfinger"/>
     </xacro:macro>
 </robot>

File: franka_description/robots/panda_arm.xacro (robot description, xacro)
@@ -285,5 +285,5 @@
       </xacro:arm_link>
     </xacro:if>
-    <!-- Empty content must be passed as block parameters cannot be defaulted-->
+    <!-- Empty content must be passed for cylinder_collision_model as block parameters cannot be defaulted-->
     <xacro:unless value="${use_cylinder_collision_model}">
       <xacro:arm_link name="${arm_id}_link0" visual_mesh="package://${description_pkg}/meshes/visual/link0.dae"
